File: CANIO.sch (EAGLE design)
At the start: 22 parts, among them T1 BT136

Commit message: Adding timer555
Configuración monoastable
R=36K
C= 10uF
t= 3.6s (aprox)
Parts:
- added C4: 0.01u, rcl:CPOL-EUB45181A
- added C5: 100u, rcl:CPOL-EUB45181A
- added IC1: LM555N, linear:LM555N
- added OK2: 4N25M, optocoupler:4N25M
- added R7: 10k, resistor:R-EU_0204/7
- added R8: 36k, resistor:R-EU_0204/7
- added R9: 220, resistor:R-EU_0204/7
Connections:
- new net N$11: IC1.TR, OK2.COL, R7.1
- new net N$15: C4.+, IC1.CV
- new net N$16: C5.+, IC1.DIS, IC1.THR, R8.1
- new net N$17: OK1.A, R9.2
- new net N$18: IC1.Q, R9.1
- net GND: now also C4.-, C5.-, IC1.GND, OK1.C, OK2.EMI
- net N$7: now also OK2.C; no longer OK1.C
- net N$8: now also OK2.A; no longer OK1.A
- net VCC: now also IC1.R, IC1.V+, R7.2, R8.2
Other:
- note added: "MAIN:"
- note added: "MONOASTABLE"
- note added: "THIS BRANCH IS:"
- note added: "TIME: 3.6s"
- note added: "TIMING"
- moved on the sheet: C2, C3, EV-1, EV-2, OK1, PS-1, PS-2, R4, R5, R6, T1
